File: Dyno22.sch (KiCad schematic (older format))
At the start: 14 parts, among them J1 Optical Sensor, J2 Power, J3 Force Sensor, J4 Brake Module, J5 I2C, U1 LM321

Commit message: Uploading changes to PCB and Schematic
* Removed button pull down resistors
* Updated rotary encoder and potentiometer footprints
* Moved display (and minor layout changes of other components)
* Added mounting holes to support rotary encoder
Parts:
- added A?: SC0918, Raspberry Pi:MODULE_SC0918, symbol Raspberry_Pi_Pico_W_SC0918:SC0918
